Commit message: Scout robot simülasyonu ve haritalama ayarlari tamamlandi

File: ugv_gazebo_sim/scout/scout_description/urdf/scout_sensors.xacro (robot description, xacro)
@@ -39,5 +39,5 @@
     <xacro:property name="front_laser_offset_x" value="0.4" />
     <xacro:property name="front_laser_offset_y" value="0.0" />
-    <xacro:property name="front_laser_offset_z" value="0.22" />
+    <xacro:property name="front_laser_offset_z" value="0.13" />
     <link name="front_laser_link">
         <visual>
@@ -67,5 +67,5 @@
     <xacro:property name="rear_laser_offset_x" value="-0.4" />
     <xacro:property name="rear_laser_offset_y" value="0.0" />
-    <xacro:property name="rear_laser_offset_z" value="0.22" />
+    <xacro:property name="rear_laser_offset_z" value="0.13" />
     <link name="rear_laser_link">
         <visual>
